Commit message: more updates; mostly working

File: ur_e_description/urdf/ur5e_joint_limited_robot.urdf.xacro (robot description, xacro)
@@ -31,5 +31,5 @@
   <xacro:include filename="$(find robotiq_85_description)/urdf/robotiq_85_gripper.urdf.xacro" />
   <xacro:robotiq_85_gripper prefix="" parent="tool_changer_tool0" >
-    <origin xyz="0.0 0.0 0.0" rpy="0.0 ${-pi/2} 0.0" />
+    <origin xyz="0.0 0.0 0.0" rpy="0.0 ${-pi/2} ${pi/2}" />
   </xacro:robotiq_85_gripper>
 </robot>

File: ur_e_description/urdf/ur5e_robot.urdf.xacro (robot description, xacro)
@@ -23,5 +23,5 @@
   <xacro:include filename="$(find robotiq_85_description)/urdf/robotiq_85_gripper.urdf.xacro" />
   <xacro:robotiq_85_gripper prefix="" parent="tool_changer_tool0" >
-    <origin xyz="0.0 0.0 0.0" rpy="0.0 ${-pi/2} 0.0" />
+    <origin xyz="0.0 0.0 0.0" rpy="0.0 ${-pi/2} ${pi/2}" />
   </xacro:robotiq_85_gripper>
 </robot>

Commit message: added table to URDF

File: ur_e_description/urdf/ur5e_joint_limited_robot.urdf.xacro (robot description, xacro)
@@ -19,7 +19,8 @@
     kinematics_file="${load_yaml('$(arg kinematics_config)')}"
   />
-  <link name="world" />
-  <joint name="world_joint" type="fixed">
-    <parent link="world" />
+  <!-- table -->
+  <xacro:include filename="$(find ur_e_description)/urdf/table.urdf.xacro" />
+  <joint name="table_joint" type="fixed">
+    <parent link="table_robot_mount_link" />
     <child link = "base_link" />
     <origin xyz="0.0 0.0 0.0" rpy="0.0 0.0 0.0" />

File: ur_e_description/urdf/ur5e_robot.urdf.xacro (robot description, xacro)
@@ -11,7 +11,8 @@
     kinematics_file="${load_yaml('$(arg kinematics_config)')}"
     />
-  <link name="world" />
-  <joint name="world_joint" type="fixed">
-    <parent link="world" />
+  <!-- table -->
+  <xacro:include filename="$(find ur_e_description)/urdf/table.urdf.xacro" />
+  <joint name="table_joint" type="fixed">
+    <parent link="table_robot_mount_link" />
     <child link = "base_link" />
     <origin xyz="0.0 0.0 0.0" rpy="0.0 0.0 0.0" />
